File: schematics/85programmer.brd (EAGLE design)
At the start: 69.5 x 53.3 mm, 3 parts, among them U1 ATTINY85-20PU

Commit message: Add capacitor value to schematics
Parts:
- C1: value (none) -> 10uF
Changed lines of the file:
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@@
 <attribute name="OC_FARNELL" value="1455162" x="102.87" y="58.42" size="1.778" layer="27" rot="R90" display="off"/>
 </element>
-<element name="C1" library="rcl" package="E2,5-6E" value="" x="31.75" y="11.43" rot="R180"/>
+<element name="C1" library="rcl" package="E2,5-6E" value="10uF" x="31.75" y="11.43" rot="R180"/>
 </elements>
 <signals>
