File: schematics/85programmer.sch (EAGLE design)
At the start: 3 parts, among them U1 ATTINY85-20PU

Commit message: Add capacitor value to schematics
Parts:
- C1: value (none) -> 10uF
Changed lines of the file:
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@@
 <part name="U$1" library="adafruit" deviceset="ARDUINO" device="UNO"/>
 <part name="U1" library="Atmel_By_element14_Batch_1-00" deviceset="ATTINY85-20PU" device=""/>
-<part name="C1" library="rcl" deviceset="CPOL-US" device="E2,5-6E"/>
+<part name="C1" library="rcl" deviceset="CPOL-US" device="E2,5-6E" value="10uF"/>
 <part name="SUPPLY1" library="supply2" deviceset="GND" device=""/>
 <part name="SUPPLY2" library="supply2" deviceset="GND" device=""/>
